File: i386/fpga-gw2ar18/hw/i386sx-gw2ar18.kicad_pcb (KiCad board)
At the start: 6 copper layers, 75 x 63.4 mm, 129 parts, among them J1 HR911105A, J2 PJ-063AH 12V, J4 SPI ISP, U1 NG80386SX-20, U100 GW2AR-LV18QN88C8/I7, U11 SN74LVC8T245PWR, U12 SN74LVC8T245PWR, U13 SN74LVC8T245PWR, U14 SN74LVC8T245PWR, U15 SN74LVC8T245PWR, U16 SN74LVC8T245PWR, U2 SN74AHCT1G125DBVR, U5 W25Q64FVDAIG (DIP-8, socketed), U6 LAN8720A-CP-TR, U7 TPS5430DDAR 12->5V, U8 TPS54620RGYR 12->3V3, U9 TPS62130RGTR VCCINT, Y1 25MHz XO, Y2 25MHz

Commit message: Publish the motherboards' KiCad files
From socket3@df617bd socket7@87d0072 socket370@615c2da i386@dcffc60
Parts:
- removed R222: 10k 1%, R_0402_1005Metric
- added J3: JTAG, PinHeader_2x05_P2.54mm_Vertical, F.Cu at (57.4, 43.9)
- added J5: UART, PinHeader_1x03_P2.54mm_Vertical, F.Cu at (57.4, 47.8)
- added R230: 1k 1%, R_0402_1005Metric, B.Cu at (75.3, 72.2)
- added R231: 1k 1%, R_0402_1005Metric, B.Cu at (76.0, 45.8)
- added R232: 4.7k 1%, R_0402_1005Metric, B.Cu at (91.2, 42.1)
- added R233: 4.7k 1%, R_0402_1005Metric, B.Cu at (88.3, 42.4)
- added R234: 1k 1%, R_0402_1005Metric, B.Cu at (110.5, 51.5)
- added R235: 1k 1%, R_0402_1005Metric, B.Cu at (112.0, 52.8)
- added R236: 4.7k 1%, R_0402_1005Metric, B.Cu at (72.1, 43.6)
- U100: value GW2AR-LV18QN88C8/I7 -> GW2AR-LV18EQ144C8/I7; footprint GW2AR-LV18QN88C8_I7 -> GW2AR-LV18EQ144C8_I7
- moved C239 24.2 mm to (93.9, 69.8)
- moved R228 21.3 mm to (115.0, 55.8)
- moved R220 19.6 mm to (97.0, 69.0), turned to 0 degrees
- moved R223 16.1 mm to (90.0, 42.4)
- moved C207 15.7 mm to (84.7, 75.5)
- moved C235 14.5 mm to (91.2, 69.3)
- moved C208 12.8 mm to (83.9, 77.7)
- moved R224 12.6 mm to (76.3, 50.4)
- moved R221 12.0 mm to (75.8, 48.0)
- moved C238 11.3 mm to (93.3, 68.6)
- moved C209 10.8 mm to (88.2, 75.3)
- moved U100 1.42 mm to (88.9, 55.4), turned to -90 degrees
Connections:
- R221 pad 1: cpu_ready_n -> fpga_mode0
- R223 pad 1: fpga_nstatus -> fpga_reconfig_n
- R224 pad 1: fpga_ads_n -> fpga_mode1
- U1 pad 4: GND -> cpu_hold
- U100 pad 10: fpga_a[15] -> fpga_a[3]
- U100 pad 11: fpga_a[16] -> fpga_a[4]
- U100 pad 12: +3V3 -> fpga_a[5]
- U100 pad 13: fpga_d[0] -> jtag_tms
- U100 pad 14: VCCINT -> jtag_tck
- U100 pad 15: fpga_d[3] -> (no net)
- U100 pad 16: fpga_d[5] -> jtag_tdi
- U100 pad 17: fpga_d[7] -> GND
- U100 pad 18: fpga_d[8] -> jtag_tdo
- U100 pad 19: fpga_d[10] -> +3V3
- U100 pad 20: fpga_d[11] -> fpga_reconfig_n
- U100 pad 21: GND -> fpga_done
- U100 pad 22: VCCINT -> fpga_ready
- U100 pad 23: +3V3 -> fpga_a[6]
- U100 pad 24: GND -> fpga_a[7]
- U100 pad 25: fpga_d[14] -> cpu_intr
- U100 pad 26: fpga_d[15] -> cpu_nmi
- U100 pad 27: fpga_xlat_dir -> fpga_a[8]
- U100 pad 28: eth_rmii_rxd[1] -> cpu_reset
- U100 pad 29: eth_rmii_rx_er -> fpga_a[9]
- U100 pad 3: +3V3 -> (no net)
- U100 pad 30: eth_rmii_crs_dv -> fpga_lock_n
- U100 pad 31: fpga_a[23] -> +3V3
- U100 pad 32: fpga_a[22] -> fpga_wr_n
- U100 pad 33: fpga_a[21] -> fpga_dc_n
- U100 pad 34: eth_ref_clk -> cpu_na_n
- U100 pad 35: clk25 -> fpga_mio_n
- U100 pad 36: fpga_a[19] -> VCCINT
- U100 pad 37: fpga_a[18] -> +3V3
- U100 pad 38: eth_rmii_tx_en -> fpga_bhe_n
- U100 pad 39: fpga_clk2 -> cpu_hold
- U100 pad 4: fpga_a[10] -> (no net)
- U100 pad 40: eth_rmii_txd[0] -> fpga_a[1]
- U100 pad 41: eth_rmii_txd[1] -> fpga_ble_n
- U100 pad 42: fpga_a[20] -> fpga_ads_n
- U100 pad 43: GND -> fpga_a[10]
- U100 pad 44: +3V3 -> fpga_a[11]
- U100 pad 45: VCCINT -> fpga_a[12]
- U100 pad 46: GND -> cpu_ready_n
- U100 pad 47: fpga_extr -> fpga_a[13]
- U100 pad 48: eth_rmii_rxd[0] -> fpga_a[14]
- U100 pad 49: fpga_d[13] -> fpga_a[15]
- U100 pad 5: fpga_a[11] -> +3V3
- U100 pad 50: VCCINT -> fpga_xlat_oe_n
- U100 pad 51: fpga_d[12] -> fpga_a[16]
- U100 pad 52: fpga_d[4] -> fpga_a[17]
- U100 pad 53: fpga_d[2] -> GND
- U100 pad 54: fpga_d[1] -> fpga_d[0]
- U100 pad 55: fpga_a[17] -> +3V3
- U100 pad 56: fpga_d[9] -> eth_ref_clk
- U100 pad 57: fpga_d[6] -> fpga_d[1]
- U100 pad 58: +3V3 -> fpga_d[2]
- U100 pad 59: spi_clk -> fpga_d[3]
- U100 pad 6: fpga_a[12] -> (no net)
- U100 pad 60: spi_cs_n -> fpga_d[4]
- U100 pad 61: spi_mosi -> fpga_d[5]
- U100 pad 62: spi_miso -> fpga_d[6]
- U100 pad 63: fpga_a[13] -> fpga_d[7]
- U100 pad 64: +3V3 -> fpga_d[8]
- U100 pad 65: GND -> fpga_d[9]
- U100 pad 66: VCCINT -> fpga_d[10]
- U100 pad 67: +3V3 -> fpga_d[11]
- U100 pad 68: GND -> fpga_d[12]
- U100 pad 69: fpga_a[2] -> fpga_d[13]
- U100 pad 7: fpga_nstatus -> (no net)
- U100 pad 70: cpu_intr -> fpga_d[14]
- U100 pad 71: cpu_nmi -> fpga_d[15]
- U100 pad 72: fpga_a[3] -> fpga_xlat_dir
- U100 pad 73: cpu_reset -> VCCINT
- U100 pad 74: fpga_a[4] -> GND
- U100 pad 75: fpga_a[5] -> fpga_extr
- U100 pad 76: fpga_a[6] -> (no net)
- U100 pad 77: fpga_a[7] -> +3V3
- U100 pad 78: +3V3 -> eth_rmii_rxd[0]
- U100 pad 79: fpga_wr_n -> eth_rmii_rx_er
- U100 pad 8: fpga_xlat_oe_n -> VCCINT
- U100 pad 80: fpga_a[8] -> eth_rmii_crs_dv
- U100 pad 81: fpga_dc_n -> VCCINT
- U100 pad 82: fpga_mio_n -> eth_mdio
- U100 pad 83: fpga_a[9] -> eth_mdc
- U100 pad 84: fpga_bhe_n -> eth_rst_n
- U100 pad 85: fpga_a[1] -> (no net)
- U100 pad 86: fpga_ble_n -> eth_rmii_rxd[1]
- U100 pad 87: fpga_ads_n -> (no net)
- U100 pad 88: cpu_ready_n -> (no net)
- U100 pad 9: fpga_a[14] -> fpga_a[2]
- U6 pad 12: +3V3 -> eth_mdio
- U6 pad 13: GND -> eth_mdc
- U7 pad 5: (no net) -> cpu_pwr_en
Routing:
- net cpu_hold: track 0.00 -> 42.2 mm, vias 0 -> 5
- net fpga_xlat_oe_n: track 95.9 -> 57.3 mm, vias 7 -> 10
- net +5V: track 208.7 -> 174.3 mm, vias 26 -> 41
- net eth_mdio: track 0.00 -> 33.2 mm, vias 0 -> 6
- net fpga_d[2]: track 60.9 -> 28.9 mm
- net GND: track 301.5 -> 269.9 mm, vias 71 -> 114
- net jtag_tck: track 0.00 -> 31.5 mm
- net jtag_tdo: track 0.00 -> 29.9 mm, vias 0 -> 1
- net eth_mdc: track 0.00 -> 28.3 mm, vias 0 -> 5
- net fpga_lock_n: track 0.00 -> 28.0 mm, vias 0 -> 2
- net eth_rst_n: track 0.00 -> 27.8 mm, vias 0 -> 1
- net fpga_hlda: track 0.66 -> 27.7 mm, vias 0 -> 4
- net fpga_d[12]: track 43.9 -> 18.3 mm, vias 2 -> 4
- net jtag_tms: track 0.00 -> 24.8 mm, vias 0 -> 1
- net cpu_pwr_en: track 0.00 -> 23.6 mm, vias 0 -> 3
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- added copper zone on In3.Cu, net VCCINT
